Commit message: Modify description for omo r1mini

File: omo_r1mini_gazebo/sdf/custom_omo_r1mini.gazebo.xacro (robot description, xacro)
@@ -1,5 +1,5 @@
 <?xml version="1.0"?>
 <robot name="omo_r1_sim" xmlns:xacro="http://ros.org/wiki/xacro">
-  <xacro:include filename="$(find omo_r1mini_gazebo)/sdf/omo_r1mini.gazebo.xacro"/>
+  <xacro:include filename="$(find omo_r1mini_gazebo)/sdf/omo_r1mini_v1.gazebo.xacro"/>
   <!-- Insert GPS Mount -->
 <!--  <link name="GPS_mount_link">-->
@@ -24,5 +24,5 @@
     <origin xyz="0 0 0" rpy="0 0 0" />
     <geometry>
-      <mesh filename="package://omo_r1mini_description/meshes/novatel-smart6.stl " scale="0.1 0.1 0.1"/>
+      <mesh filename="package://omo_r1mini_description/meshes/novatel-smart6.stl" scale="0.1 0.1 0.1"/>
     </geometry>
     <material name="novatel_white">
@@ -32,7 +32,8 @@
   </link>
   <joint name="GPS_joint" type="fixed">
-    <parent link="base_link" />
+    <parent link="base_footprint" />
     <child link="GPS_link" />
-    <origin xyz="-0.1 0 0.01" rpy="0 0 0" />
+<!--    <origin xyz="-0.1 0 0.01" rpy="0 0 0" />-->
+    <origin xyz="-0.1 0 0.0435" rpy="0 0 0" />
   </joint>
 </robot>
