Commit message: Change parent frame of all sensors to base_link

File: omo_r1mini_description/urdf/r1mini_v1.urdf.xacro (robot description, xacro)
@@ -141,5 +141,5 @@
   </link>
   <joint name="imu_joint" type="fixed">
-    <parent link="base_footprint"/>
+    <parent link="base_link"/>
     <child link="imu_link"/>
 <!--    <origin xyz="0.0 0 0.038" rpy="0 0 0"/>-->

File: omo_r1mini_gazebo/sdf/custom_omo_r1mini.gazebo.xacro (robot description, xacro)
@@ -32,8 +32,7 @@
   </link>
   <joint name="GPS_joint" type="fixed">
-    <parent link="base_footprint" />
+    <parent link="base_link" />
     <child link="GPS_link" />
-<!--    <origin xyz="-0.1 0 0.01" rpy="0 0 0" />-->
-    <origin xyz="-0.1 0 0.0435" rpy="0 0 0" />
+    <origin xyz="-0.1 0 0.01" rpy="0 0 0" />
   </joint>
 </robot>

File: omo_r1mini_gazebo/sdf/omo_r1mini_v1.gazebo.xacro (robot description, xacro)
@@ -36,5 +36,4 @@
       <odometrySource>world</odometrySource>
       <publishOdomTF>true</publishOdomTF>
-<!--      <robotBaseFrame>base_link</robotBaseFrame>-->
       <robotBaseFrame>base_footprint</robotBaseFrame>
       <publishWheelTF>false</publishWheelTF>
@@ -55,6 +54,5 @@
     <plugin name="imu_controller" filename="libgazebo_ros_imu.so">
       <alwaysOn>true</alwaysOn>
-<!--      <bodyName>base_link</bodyName>-->
-      <bodyName>base_footprint</bodyName>
+      <bodyName>base_link</bodyName>
       <frameName>imu_link</frameName>
       <topicName>imu/data</topicName>
@@ -152,6 +150,6 @@
     <plugin name="gps_controller" filename="libhector_gazebo_ros_gps.so">
       <updateRate>40</updateRate>
-      <bodyName>base_footprint</bodyName>
-      <frameId>base_footprint</frameId>
+      <bodyName>base_link</bodyName>
+      <frameId>base_link</frameId>
       <topicName>navsat/fix</topicName>
       <velocityTopicName>navsat/vel</velocityTopicName>

Commit message: Modify URDF file of omo r1mini

File: omo_r1mini_description/urdf/r1mini_v1.urdf.xacro (robot description, xacro)
@@ -1,182 +1,197 @@
 <?xml version="1.0" ?>
 <robot name="r1mini" xmlns:xacro="http://ros.org/wiki/xacro">
-  <xacro:include filename="$(find omo_r1mini_description)/urdf/common_properties.xacro"/>
-  <link name="base_footprint"/>
-  <joint name="base_footprint_joint" type="fixed">
-    <parent link="base_footprint"/>
-    <child link="base_link" />
-    <origin xyz="0 0 0.0335" rpy="0 0 0.0"/>
-  </joint>
-  <link name="base_link">
-    <visual>
-      <origin xyz="0.03 -0.065 -0.022" rpy="0 0 1.5707963"/>
-      <geometry>
-        <mesh filename="package://omo_r1mini_description/meshes/bases/mini_frame.stl" scale="0.001 0.001 0.001"/>
-      </geometry>
-      <material name="dark"/>
-    </visual>
-    <collision>
-      <origin xyz="0.03 -0.065 -0.022" rpy="0 0 1.5707963"/>
-      <geometry>
-        <mesh filename="package://omo_r1mini_description/meshes/bases/mini_frame.stl" scale="0.001 0.001 0.001"/>
-      </geometry>
-    </collision>
-    <inertial>
-      <origin xyz="-0.01 0 0" rpy="0 0 0"/>
-      <mass value="1.3729096e+00"/>
-      <inertia ixx="8.7002718e-03" ixy="-4.7576583e-05" ixz="1.1160499e-04"
-               iyy="8.6195418e-03" iyz="-3.5422299e-06"
-               izz="1.4612727e-02" />
-      </inertial>
-  </link>
-  <joint name="housing_joint" type="fixed">
-    <parent link="base_link"/>
-    <child link="housing_link" />
-    <origin xyz="0 0 0" rpy="0 0 0.0"/>
-  </joint>
-  <link name="housing_link">
-    <visual>
-      <origin xyz="-0.028 0 -0.028" rpy="0 0 1.5707963"/>
-      <geometry>
-        <mesh filename="package://omo_r1mini_description/meshes/bases/r1mini housing lite 2.stl" scale="0.001 0.001 0.001"/>
-      </geometry>
-      <material name="pink"/>
-    </visual>
-    <collision>
-      <origin xyz="-0.028 0 -0.028" rpy="0 0 1.5707963"/>
-      <geometry>
-        <mesh filename="package://omo_r1mini_description/meshes/bases/r1mini housing lite 2.stl" scale="0.001 0.001 0.001"/>
-      </geometry>
-    </collision>
-    <inertial>
-      <origin xyz="-0.1 0 0" rpy="0 0 0"/>
-      <mass value="0.01"/>
-      <inertia ixx="8.7002718e-04" ixy="-4.7576583e-07" ixz="1.1160499e-07"
-               iyy="8.6195418e-04" iyz="-3.5422299e-07"
-               izz="1.4612727e-04" />
-    </inertial>
-  </link>
-  <joint name="wheel_left_joint" type="continuous">
-    <parent link="base_link"/>
-    <child link="wheel_left_link"/>
-    <origin xyz="0.0 0.096 0.0" rpy="0.0 0.0 0"/>
-    <axis xyz="0 1 0"/>
-  </joint>
-  <link name="wheel_left_link">
-    <visual>
-      <origin xyz="-0.0335 -0.004 -0.0335" rpy="1.5707963 0 0"/>
-      <geometry>
-        <mesh filename="package://omo_r1mini_description/meshes/wheels/mini_tire.stl" scale="0.001 0.001 0.001"/>
-      </geometry>
-      <material name="dark"/>
-    </visual>
-    <collision>
-      <origin xyz="-0.0335 -0.004 -0.0335" rpy="1.5707963 0 0"/>
-      <geometry>
-        <mesh filename="package://omo_r1mini_description/meshes/wheels/mini_tire.stl" scale="0.001 0.001 0.001"/>
-      </geometry>
-    </collision>
-    <inertial>
-      <origin xyz="0 -0.01675 0" rpy="-1.5707963 0 0" />
-      <mass value="2.8498940e-02" />
-      <inertia ixx="1.1175580e-05" ixy="0" ixz="0"
-               iyy="1.1192413e-05" iyz="0"
-               izz="2.0712558e-05" />
-    </inertial>
-  </link>
-  <joint name="wheel_right_joint" type="continuous">
-    <parent link="base_link"/>
-    <child link="wheel_right_link"/>
-    <origin xyz="0.0 -0.096 0.0" rpy="0.0 0.0 0"/>
-    <axis xyz="0 1 0"/>
-  </joint>
-  <link name="wheel_right_link">
-    <visual>
-      <origin xyz="-0.0335 0.004 0.0335" rpy="-1.5707963 0 0"/>
-      <geometry>
-        <mesh filename="package://omo_r1mini_description/meshes/wheels/mini_tire.stl" scale="0.001 0.001 0.001"/>
-      </geometry>
-      <material name="dark"/>
-    </visual>
-    <collision>
-      <origin xyz="-0.0335 0.004 0.0335" rpy="-1.5707963 0 0"/>
-      <geometry>
-        <mesh filename="package://omo_r1mini_description/meshes/wheels/mini_tire.stl" scale="0.001 0.001 0.001"/>
-      </geometry>
-    </collision>
-    <inertial>
-      <origin xyz="0 0.01675 0" rpy="-1.5707963 0 0" />
-      <mass value="2.8498940e-02" />
-      <inertia ixx="1.1175580e-05" ixy="0" ixz="0"
-               iyy="1.1192413e-05" iyz="0"
-               izz="2.0712558e-05" />
-    </inertial>
-  </link>
-  <joint name="caster_back_joint" type="fixed">
-    <parent link="base_link"/>
-    <child link="caster_back_link"/>
-    <origin xyz="-0.12 0.0 -0.018" rpy="0 0 0"/>
-  </joint>
-  <link name="caster_back_link">
-    <visual>
-      <origin xyz="-0.016 -0.007 -0.016" rpy="0 0 0"/>
-      <geometry>
-        <mesh filename="package://omo_r1mini_description/meshes/wheels/mini_caster.stl" scale="0.001 0.001 0.001"/>
-      </geometry>
-      <material name="dark"/>
-    </visual>
-    <collision>
-      <origin xyz="-0.016 -0.007 -0.016" rpy="0 0 0"/>
-      <geometry>
-        <mesh filename="package://omo_r1mini_description/meshes/wheels/mini_caster.stl" scale="0.001 0.001 0.001"/>
-      </geometry>
-    </collision>
-    <inertial>
-      <origin xyz="0 0 0" />
-      <mass value="0.005" />
-      <inertia ixx="0.001" ixy="0.0" ixz="0.0"
-               iyy="0.001" iyz="0.0"
-               izz="0.001" />
-    </inertial>
-  </link>
-  <joint name="imu_joint" type="fixed">
-    <parent link="base_link"/>
-    <child link="imu_link"/>
-<!--    <origin xyz="0.0 0 0.038" rpy="0 0 0"/>-->
-    <origin xyz="0.0 0 0.0715" rpy="0 0 0"/>
-  </joint>
-  <link name="imu_link"/>
-  <joint name="scan_joint" type="fixed">
-    <parent link="base_link"/>
-    <child link="base_scan"/>
-    <origin xyz="0.0 0 0.07" rpy="0.0 0 3.14159"/>
-  </joint>
-  <link name="base_scan">
-    <visual>
-      <origin xyz="0 0 0.0" rpy="0 0 0"/>
-      <geometry>
-        <mesh filename="package://omo_r1mini_description/meshes/sensors/lds.stl" scale="0.001 0.001 0.001"/>
-      </geometry>
-      <material name="dark"/>
-    </visual>
-    <collision>
-      <origin xyz="0.015 0 -0.0065" rpy="0 0 0"/>
-      <geometry>
-        <cylinder length="0.0315" radius="0.055"/>
-      </geometry>
-    </collision>
-    <inertial>
-      <mass value="0.05" />
-      <origin xyz="0 0 0" />
-      <inertia ixx="0.001" ixy="0.0" ixz="0.0"
-               iyy="0.001" iyz="0.0"
-               izz="0.001" />
-    </inertial>
-  </link>
-  <joint name="camera_joint" type="fixed">
-    <origin xyz="0.04 0 0.02" rpy="3.14159 -1.570796 0"/>
-    <parent link="base_link"/>
-    <child link="main_camera_optical"/>
-  </joint>
-  <link name="main_camera_optical"/>
+    <xacro:include filename="$(find omo_r1mini_description)/urdf/common_properties.xacro"/>
+    <link name="base_footprint"/>
+    <joint name="base_joint" type="fixed">
+        <parent link="base_footprint"/>
+        <child link="base_link"/>
+        <origin xyz="0 0 0.0335" rpy="0 0 0.0"/>
+    </joint>
+    <link name="base_link">
+        <visual>
+            <origin xyz="0.03 -0.065 -0.022" rpy="0 0 1.57"/>
+            <geometry>
+                <mesh filename="package://omo_r1mini_description/meshes/bases/mini_frame.stl"
+                      scale="0.001 0.001 0.001"/>
+            </geometry>
+            <material name="dark"/>
+        </visual>
+        <collision>
+            <origin xyz="0.03 -0.065 -0.022" rpy="0 0 1.57"/>
+            <geometry>
+                <mesh filename="package://omo_r1mini_description/meshes/bases/mini_frame.stl"
+                      scale="0.001 0.001 0.001"/>
+            </geometry>
+        </collision>
+        <inertial>
+            <origin xyz="-0.1 0 0" rpy="0 0 0"/>
+            <mass value="1.3729096e+00"/>
+            <inertia ixx="8.7002718e-03" ixy="-4.7576583e-05" ixz="1.1160499e-04"
+                     iyy="8.6195418e-03" iyz="-3.5422299e-06"
+                     izz="1.4612727e-02"/>
+        </inertial>
+    </link>
+    <joint name="housing_joint" type="fixed">
+        <parent link="base_link"/>
+        <child link="housing_link"/>
+        <origin xyz="0 0 0" rpy="0 0 0.0"/>
+    </joint>
+    <link name="housing_link">
+        <visual>
+            <origin xyz="-0.028 0 -0.028" rpy="0 0 1.57"/>
+            <geometry>
+                <mesh filename="package://omo_r1mini_description/meshes/bases/r1mini housing lite 2.stl"
+                      scale="0.001 0.001 0.001"/>
+            </geometry>
+            <material name="pink"/>
+        </visual>
+        <collision>
+            <origin xyz="-0.028 0 -0.028" rpy="0 0 1.57"/>
+            <geometry>
+                <mesh filename="package://omo_r1mini_description/meshes/bases/r1mini housing lite 2.stl"
+                      scale="0.001 0.001 0.001"/>
+            </geometry>
+        </collision>
+        <inertial>
+            <origin xyz="-0.1 0 0" rpy="0 0 0"/>
+            <mass value="0.01"/>
+            <inertia ixx="8.7002718e-04" ixy="-4.7576583e-07" ixz="1.1160499e-07"
+                     iyy="8.6195418e-04" iyz="-3.5422299e-07"
+                     izz="1.4612727e-04"/>
+        </inertial>
+    </link>
+    <joint name="wheel_left_joint" type="continuous">
+        <parent link="base_link"/>
+        <child link="wheel_left_link"/>
+        <origin xyz="0.0 0.096 0.0" rpy="0.0 0.0 0"/>
+        <axis xyz="0 1 0"/>
+    </joint>
+    <link name="wheel_left_link">
+        <visual>
+            <origin xyz="-0.0335 -0.004 -0.0335" rpy="1.57 0 0"/>
+            <geometry>
+                <mesh filename="package://omo_r1mini_description/meshes/wheels/mini_tire.stl"
+                      scale="0.001 0.001 0.001"/>
+            </geometry>
+            <material name="dark"/>
+        </visual>
+        <collision>
+            <origin xyz="-0.0335 -0.004 -0.0335" rpy="1.57 0 0"/>
+            <geometry>
+                <mesh filename="package://omo_r1mini_description/meshes/wheels/mini_tire.stl"
+                      scale="0.001 0.001 0.001"/>
+            </geometry>
+        </collision>
+        <inertial>
+            <origin xyz="0 0 0"/>
+            <mass value="2.8498940e-02"/>
+            <inertia ixx="1.1175580e-05" ixy="-4.2369783e-11" ixz="-5.9381719e-09"
+                     iyy="1.1192413e-05" iyz="-1.4400107e-11"
+                     izz="2.0712558e-05"/>
+        </inertial>
+    </link>
+    <joint name="wheel_right_joint" type="continuous">
+        <parent link="base_link"/>
+        <child link="wheel_right_link"/>
+        <origin xyz="0.0 -0.096 0.0" rpy="0.0 0.0 0"/>
+        <axis xyz="0 1 0"/>
+    </joint>
+    <link name="wheel_right_link">
+        <visual>
+            <origin xyz="-0.0335 0.004 0.0335" rpy="-1.57 0 0"/>
+            <geometry>
+                <mesh filename="package://omo_r1mini_description/meshes/wheels/mini_tire.stl"
+                      scale="0.001 0.001 0.001"/>
+            </geometry>
+            <material name="dark"/>
+        </visual>
+        <collision>
+            <origin xyz="-0.0335 0.004 0.0335" rpy="-1.57 0 0"/>
+            <geometry>
+                <mesh filename="package://omo_r1mini_description/meshes/wheels/mini_tire.stl"
+                      scale="0.001 0.001 0.001"/>
+            </geometry>
+        </collision>
+        <inertial>
+            <origin xyz="0 0 0"/>
+            <mass value="2.8498940e-02"/>
+            <inertia ixx="1.1175580e-05" ixy="-4.2369783e-11" ixz="-5.9381719e-09"
+                     iyy="1.1192413e-05" iyz="-1.4400107e-11"
+                     izz="2.0712558e-05"/>
+        </inertial>
+    </link>
+    <joint name="caster_back_joint" type="fixed">
+        <parent link="base_link"/>
+        <child link="caster_back_link"/>
+        <origin xyz="-0.12 0.0 -0.018" rpy="0 0 0"/>
+    </joint>
+    <link name="caster_back_link">
+        <visual>
+            <origin xyz="-0.016 -0.007 -0.016" rpy="0 0 0"/>
+            <geometry>
+                <mesh filename="package://omo_r1mini_description/meshes/wheels/mini_caster.stl"
+                      scale="0.001 0.001 0.001"/>
+            </geometry>
+            <material name="dark"/>
+        </visual>
+        <collision>
+            <origin xyz="-0.016 -0.007 -0.016" rpy="0 0 0"/>
+            <geometry>
+                <mesh filename="package://omo_r1mini_description/meshes/wheels/mini_caster.stl"
+                      scale="0.001 0.001 0.001"/>
+            </geometry>
+        </collision>
+        <inertial>
+            <origin xyz="0 0 0"/>
+            <mass value="0.005"/>
+            <inertia ixx="0.001" ixy="0.0" ixz="0.0"
+                     iyy="0.001" iyz="0.0"
+                     izz="0.001"/>
+        </inertial>
+    </link>
+    <joint name="imu_joint" type="fixed">
+        <parent link="base_link"/>
+        <child link="imu_link"/>
+        <origin xyz="0.0 0 0.0715" rpy="0 0 0"/>
+    </joint>
+    <link name="imu_link"/>
+    <joint name="scan_joint" type="fixed">
+        <parent link="base_link"/>
+        <child link="base_scan"/>
+        <origin xyz="0.0 0 0.07" rpy="0.0 0 3.14159"/>
+    </joint>
+    <link name="base_scan">
+        <visual>
+            <origin xyz="0 0 0.0" rpy="0 0 0"/>
+            <geometry>
+                <mesh filename="package://omo_r1mini_description/meshes/sensors/lds.stl" scale="0.001 0.001 0.001"/>
+            </geometry>
+            <material name="dark"/>
+        </visual>
+        <collision>
+            <origin xyz="0.015 0 -0.0065" rpy="0 0 0"/>
+            <geometry>
+                <cylinder length="0.0315" radius="0.055"/>
+            </geometry>
+        </collision>
+        <inertial>
+            <mass value="0.05"/>
+            <origin xyz="0 0 0"/>
+            <inertia ixx="0.001" ixy="0.0" ixz="0.0"
+                     iyy="0.001" iyz="0.0"
+                     izz="0.001"/>
+        </inertial>
+    </link>
+    <joint name="camera_joint" type="fixed">
+        <origin xyz="0.04 0 0.02" rpy="3.14159 -1.570796 0"/>
+        <parent link="base_link"/>
+        <child link="main_camera_optical"/>
+    </joint>
+    <link name="main_camera_optical"/>
+    <joint name="GPS_joint" type="fixed">
+        <parent link="base_link"/>
+        <child link="GPS_link"/>
+        <origin xyz="-0.1 0 0.01" rpy="0 0 0"/>
+    </joint>
+    <link name="GPS_link"/>
 </robot>

File: omo_r1mini_gazebo/sdf/custom_omo_r1mini.gazebo.xacro (robot description, xacro)
@@ -2,37 +2,3 @@
 <robot name="omo_r1_sim" xmlns:xacro="http://ros.org/wiki/xacro">
   <xacro:include filename="$(find omo_r1mini_gazebo)/sdf/omo_r1mini_v1.gazebo.xacro"/>
-  <!-- Insert GPS Mount -->
-<!--  <link name="GPS_mount_link">-->
-<!--  <visual>-->
-<!--    <origin xyz="0 0 0" rpy="0 0 0" />-->
-<!--    <geometry>-->
-<!--      <mesh filename="package://omo_r1mini_description/meshes/gps_mount.STL" scale="0.0005 0.0005 0.0005" />-->
-<!--    </geometry>-->
-<!--    <material name="black">-->
-<!--      <color rgba="0 0 0 1.0" />-->
-<!--    </material>-->
-<!--  </visual>-->
-<!--  </link>-->
-<!--  <joint name="GPS_mount_joint" type="fixed">-->
-<!--    <parent link="base_link" />-->
-<!--    <child link="GPS_mount_link" />-->
-<!--    <origin xyz="0 0 0.1" rpy="0 0 0" />-->
-<!--  </joint>-->
-  <!-- Insert GPS -->
-  <link name="GPS_link">
-  <visual>
-    <origin xyz="0 0 0" rpy="0 0 0" />
-    <geometry>
-      <mesh filename="package://omo_r1mini_description/meshes/novatel-smart6.stl" scale="0.1 0.1 0.1"/>
-    </geometry>
-    <material name="novatel_white">
-      <color rgba="0.8 0.8 0.8 1.0" />
-    </material>
-  </visual>
-  </link>
-  <joint name="GPS_joint" type="fixed">
-    <parent link="base_link" />
-    <child link="GPS_link" />
-    <origin xyz="-0.1 0 0.01" rpy="0 0 0" />
-  </joint>
 </robot>
